File: MTA-PWM_v3/MTA-PWM_v3.kicad_pcb (KiCad board)
At the start: 2 copper layers, 95.9 x 90.2 mm, 29 parts, among them J1 Conn_02x26_Odd_Even, J2 Conn_02x26_Odd_Even, J3 2053380002, J4 2053380002, J5 532610271, Q3 NMOS, Q4 PMOS, Q5 NMOS, Q6 PMOS, Q7 NMOS, Q8 PMOS, U1 DRV8231ADDAR, U2 DRV8231ADDAR, U3 DRV8231ADDAR

Commit message: Pinout updates
Parts:
- J1, J2: footprint HSL_pc104:pc104-PinSocket_2x26_P2.54mm_Vertical -> PC104:PC140Header_2x26_P2.54mm_Vertical
- moved J2 33.5 mm to (110.9, 118.4)
- moved J1 33.4 mm to (116.1, 118.3)
- moved TP2 30.9 mm to (160.1, 113.3)
- moved U3 30.9 mm to (156.7, 50.6)
- moved H4 30.9 mm to (111.0, 49.8)
- moved H2 30.9 mm to (111.0, 123.4)
- moved J5 30.9 mm to (168.4, 50.1)
- moved MT3 30.9 mm to (173.9, 81.3)
- moved Q3 30.9 mm to (128.5, 90.1)
- moved R2 30.9 mm to (160.1, 109.8)
- moved Q5 30.9 mm to (179.7, 109.7)
- moved Q4 30.9 mm to (132.1, 90.1)
- moved Q8 30.9 mm to (129.0, 55.9)
- moved C1 30.9 mm to (124.7, 96.3)
- moved C3 30.9 mm to (124.7, 66.8)
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Connections:
- C1 pad 1: 5V_PERM -> 5V_IN
- C3 pad 1: 12V -> 12V_IN
- Q3 pad 1: ACDS_PWM_1 -> ADCS_PWM_1
- Q3 pad 2: ACDS_GPIO_1 -> ADCS_GPIO_1
- Q4 pad 2: ACDS_GPIO_1 -> ADCS_GPIO_1
- Q4 pad 3: ACDS_PWM_1 -> ADCS_PWM_1
- Q5 pad 1: ACDS_PWM_2 -> ADCS_PWM_2
- Q5 pad 2: ACDS_GPIO_2 -> ADCS_GPIO_2
- Q6 pad 2: ACDS_GPIO_2 -> ADCS_GPIO_2
- Q6 pad 3: ACDS_PWM_2 -> ADCS_PWM_2
- Q7 pad 1: ACDS_PWM_3 -> ADCS_PWM_3
- Q7 pad 2: ACDS_GPIO_3 -> ADCS_GPIO_3
- Q8 pad 2: ACDS_GPIO_3 -> ADCS_GPIO_3
- Q8 pad 3: ACDS_PWM_3 -> ADCS_PWM_3
- U1 pad 4: 3.3V -> 3.3V_IN
- U1 pad 5: 5V_PERM -> 5V_IN
- U2 pad 4: 3.3V -> 3.3V_IN
- U2 pad 5: 5V_PERM -> 5V_IN
- U3 pad 4: 3.3V -> 3.3V_IN
- U3 pad 5: 12V -> 12V_IN
Routing:
- net 5V_IN: track 0.00 -> 128.6 mm, vias 0 -> 4
- net 3.3V_IN: track 0.00 -> 128.5 mm, vias 0 -> 3
- net 3.3V: track 112.0 -> 0.00 mm, vias 3 -> 0
- net 12V_IN: track 0.00 -> 99.0 mm, vias 0 -> 1
- net 5V_PERM: track 87.5 -> 0.00 mm, vias 3 -> 0
- net ADCS_PWM_2: track 0.00 -> 85.9 mm, vias 0 -> 1
- net 12V: track 85.1 -> 0.00 mm, vias 1 -> 0
- net ACDS_PWM_2: track 84.5 -> 0.00 mm, vias 1 -> 0
- net ADCS_GPIO_2: track 0.00 -> 79.8 mm, vias 0 -> 1
- net ACDS_GPIO_2: track 75.8 -> 0.00 mm, vias 1 -> 0
- net ACDS_PWM_3: track 38.1 -> 0.00 mm, vias 2 -> 0
- net ADCS_PWM_3: track 0.00 -> 37.0 mm, vias 0 -> 1
- net ADCS_GPIO_3: track 0.00 -> 36.6 mm, vias 0 -> 1
- net ACDS_GPIO_3: track 36.4 -> 0.00 mm
- net GND: track 6.34 -> 41.0 mm
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