File: MTA-PWM_v3/MTA-PWM_v3.kicad_sch (KiCad schematic)
At the start: 23 parts, among them J1 Conn_02x26_Odd_Even, J2 Conn_02x26_Odd_Even, J3 2053380002, J4 2053380002, J5 532610271, Q3 NMOS, Q4 PMOS, Q5 NMOS, Q6 PMOS, Q7 NMOS, Q8 PMOS, U1 DRV8231ADDAR, U2 DRV8231ADDAR, U3 DRV8231ADDAR

Commit message: Pinout updates
Parts:
- J1, J2: footprint HSL_pc104:pc104-PinSocket_2x26_P2.54mm_Vertical -> PC104:PC140Header_2x26_P2.54mm_Vertical; symbol Connector_Generic:Conn_02x26_Odd_Even -> Connector_Generic:Conn_02x26_Row_Letter_First
Connections:
- net GND: now also J1.a23 (Pin_a23), J1.a25 (Pin_a25), J1.b1 (Pin_b1), J1.b10 (Pin_b10), J1.b17 (Pin_b17), J1.b23 (Pin_b23), J1.b25 (Pin_b25), J2.a11 (Pin_a11), J2.a14 (Pin_a14), J2.a15 (Pin_a15), J2.a16 (Pin_a16), J2.a22 (Pin_a22), J2.a25 (Pin_a25), J2.a6 (Pin_a6), J2.b11 (Pin_b11), J2.b14 (Pin_b14), J2.b15 (Pin_b15), J2.b16 (Pin_b16), J2.b22 (Pin_b22), J2.b25 (Pin_b25), J2.b6 (Pin_b6); no longer J1.33 (Pin_33), J1.34 (Pin_34), J2.29 (Pin_29), J2.30 (Pin_30), J2.31 (Pin_31), J2.32 (Pin_32)
- net 12V renamed 12V_IN
- net 12V_IN: now also J1.a24 (Pin_a24), J1.b24 (Pin_b24), J2.a12 (Pin_a12), J2.b12 (Pin_b12); no longer J2.23 (Pin_23), J2.24 (Pin_24)
- net 3.3V renamed 3.3V_IN
- net 3.3V_IN: now also J1.a13 (Pin_a13), J1.b13 (Pin_b13), J2.a13 (Pin_a13), J2.b13 (Pin_b13); no longer J2.27 (Pin_27), J2.28 (Pin_28)
- net 5V_PERM renamed 5V_IN
- net 5V_IN: now also J1.a26 (Pin_a26), J1.b26 (Pin_b26), J2.a26 (Pin_a26), J2.b26 (Pin_b26); no longer J1.25 (Pin_25), J1.26 (Pin_26), J2.25 (Pin_25), J2.26 (Pin_26)
- net ACDS_GPIO_1 renamed ADCS_GPIO_1
- net ADCS_GPIO_1: now also J1.a10 (Pin_a10); no longer J1.19 (Pin_19)
- net ACDS_GPIO_2 renamed ADCS_GPIO_2
- net ADCS_GPIO_2: now also J1.a12 (Pin_a12); no longer J1.23 (Pin_23)
- net ACDS_GPIO_3 renamed ADCS_GPIO_3
- net ADCS_GPIO_3: now also J1.a16 (Pin_a16); no longer J1.31 (Pin_31)
- removed net ACDS_IMU_RST: J1.30 (Pin_30)
- net ACDS_PWM_1 renamed ADCS_PWM_1
- net ADCS_PWM_1: now also J1.a9 (Pin_a9); no longer J1.17 (Pin_17)
- net ACDS_PWM_2 renamed ADCS_PWM_2
- net ADCS_PWM_2: now also J1.a11 (Pin_a11); no longer J1.21 (Pin_21)
- net ACDS_PWM_3 renamed ADCS_PWM_3
- net ADCS_PWM_3: now also J1.a15 (Pin_a15); no longer J1.29 (Pin_29)
- removed net ACDS_RS232_RX: J1.8 (Pin_8)
- removed net ACDS_RS232_TX: J1.6 (Pin_6)
- removed net BATT_PIN: J2.45 (Pin_45), J2.47 (Pin_47)
- removed net DS_A: J2.51 (Pin_51)
- removed net DS_B: J2.52 (Pin_52)
- removed net HEATER_PWM: J2.20 (Pin_20)
- removed net INT: J1.12 (Pin_12)
- removed net PG: J1.10 (Pin_10)
- removed net RBF_A: J2.49 (Pin_49)
- removed net RBF_B: J2.50 (Pin_50)
- removed net RS SYS2 Rx: J1.39 (Pin_39)
- removed net RS SYS2 Tx: J1.40 (Pin_40)
- removed net RS-485 SYS1 B: J1.22 (Pin_22), J1.24 (Pin_24)
- removed net SCL: J1.18 (Pin_18)
- removed net SDA: J1.16 (Pin_16)
- removed net SOL_PIN: J2.43 (Pin_43), J2.44 (Pin_44)
- removed net STAT_1: J1.14 (Pin_14)
- removed net STAT_2: J1.9 (Pin_9)
- removed net SUN_SENSE_1: J2.1 (Pin_1)
- removed net SUN_SENSE_2: J2.2 (Pin_2)
- removed net SUN_SENSE_3: J2.3 (Pin_3)
- removed net SUN_SENSE_4: J2.4 (Pin_4)
- removed net SYS_PIN: J2.46 (Pin_46), J2.48 (Pin_48)
- removed net THR_1: J2.5 (Pin_5)
- removed net THR_2: J2.6 (Pin_6)
- removed net THR_3: J2.7 (Pin_7)
- removed net THR_4: J2.8 (Pin_8)
- removed net THR_5: J2.10 (Pin_10)
- removed net THR_6: J2.12 (Pin_12)
- removed net THR_7: J2.14 (Pin_14)
- removed net THR_8: J2.16 (Pin_16)
- removed net THR_9: J2.18 (Pin_18)
- removed net UART_RX: J1.42 (Pin_42)
- removed net UART_TX: J1.44 (Pin_44)
- no-connect marks 45 -> 0
Other:
- moved on the sheet: J1, J2, Q3, Q4, Q5, Q6, Q7, Q8
